File: CoolPackReceiver/CoolPackReceiver.kicad_sch (KiCad schematic)
At the start: 1 part, among them U1 Si4463

Commit message: [add] KiCad Starting
Parts:
- removed U1: Si4463, Package_DFN_QFN:QFN-20-1EP_4x4mm_P0.5mm_EP2.6x2.6mm_ThermalVias, symbol RF:Si4463
- added U3: PCM5102APW, PW0020A_N, symbol CustomFootPrints:PCM5102APW
Connections:
- new net VSSA: U3.9 (AGND)
Other:
- added sheet MCU (MCU.kicad_sch)
- added sheet Power (Power.kicad_sch)
- added sheet RF sheet (RF.kicad_sch)
- note added: "DAC"

Commit message: [Update] Part Choice
Parts:
- removed U3: PCM5102APW, PW0020A_N, symbol CustomFootPrints:PCM5102APW
- added U3: PCM1796DB, DB28, symbol CustomFootPrints:PCM1796DB
Other:
- note added: "DAC TO OUTPUT"
- note removed: "DAC"
Changed lines of the file:
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@@
 	(rectangle
 		(start 22.86 86.36)
-		(end 76.2 179.07)
+		(end 102.87 179.07)
 		(stroke
 			(width 0)
@@
 		)
 	)
-	(text "DAC"
+	(text "DAC TO OUTPUT"
 		(exclude_from_sim no)
-		(at 32.004 90.678 0)
+		(at 53.594 90.678 0)
 		(effects
 			(font
@@
 		)
 	)
-	(wire
-		(pts
-			(xy 73.66 160.02) (xy 81.28 160.02)
-		)
-		(stroke
-			(width 0)
-			(type default)
-		)
-	)
 	(symbol
-		(lib_id "power:VSSA")
-		(at 81.28 160.02 180)
-		(unit 1)
-		(exclude_from_sim no)
-		(in_bom yes)
-		(on_board yes)
-		(dnp no)
-		(fields_autoplaced yes)
-		(property "Reference" "#PWR04"
-			(at 81.28 156.21 0)
-			(effects
-				(font
-					(size 1.27 1.27)
-				)
-				(hide yes)
-			)
-		)
-		(property "Value" "VSSA"
-			(at 81.28 165.1 0)
-			(effects
-				(font
-					(size 1.27 1.27)
-				)
-			)
-		)
-		(property "Footprint" ""
-			(at 81.28 160.02 0)
-			(effects
-				(font
-					(size 1.27 1.27)
-				)
-				(hide yes)
-			)
-		)
-		(property "Datasheet" ""
-			(at 81.28 160.02 0)
-			(effects
-				(font
-					(size 1.27 1.27)
-				)
-				(hide yes)
-			)
-		)
-		(property "Description" "Power symbol creates a global label with name \"VSSA\""
-			(at 81.28 160.02 0)
-			(effects
-				(font
-					(size 1.27 1.27)
-				)
-				(hide yes)
-			)
-		)
-		(pin "1"
-		)
-		(instances
-			(project ""
-				(path "/0f8c4546-fe83-48ba-bceb-d590a2a5b006"
-					(reference "#PWR04")
-					(unit 1)
-				)
-			)
-		)
-	)
-	(symbol
-		(lib_id "CustomFootPrints:PCM5102APW")
-		(at 53.34 139.7 0)
+		(lib_id "CustomFootPrints:PCM1796DB")
+		(at 29.21 110.49 0)
 		(unit 1)
 		(exclude_from_sim no)
@@
 		(fields_autoplaced yes)
 		(property "Reference" "U3"
-			(at 53.34 106.68 0)
+			(at 62.23 100.33 0)
 			(effects
 				(font
@@
 			)
 		)
-		(property "Value" "PCM5102APW"
-			(at 53.34 109.22 0)
+		(property "Value" "PCM1796DB"
+			(at 62.23 102.87 0)
 			(effects
 				(font
@@
 			)
 		)
-		(property "Footprint" "PW0020A_N"
-			(at 53.34 139.7 0)
+		(property "Footprint" "DB28"
+			(at 29.21 110.49 0)
 			(effects
 				(font
@@
 			)
 		)
-		(property "Datasheet" "https://www.ti.com/lit/gpn/pcm5102a"
-			(at 53.34 139.7 0)
+		(property "Datasheet" "https://www.ti.com/lit/gpn/pcm1796"
+			(at 29.21 110.49 0)
 			(effects
 				(font
@@
 		)
 		(property "Description" ""
-			(at 53.34 139.7 0)
+			(at 29.21 110.49 0)
 			(effects
 				(font
@@
 			)
 		)
-		(pin "2"
+		(pin "24"
+		)
+		(pin "4"
+		)
+		(pin "1"
+		)
+		(pin "27"
+		)
+		(pin "6"
+		)
+		(pin "16"
+		)
+		(pin "17"
 		)
 		(pin "7"
 		)
+		(pin "21"
+		)
 		(pin "18"
 		)
-		(pin "6"
+		(pin "15"
+		)
+		(pin "12"
+		)
+		(pin "14"
+		)
+		(pin "13"
+		)
+		(pin "8"
+		)
+		(pin "23"
+		)
+		(pin "28"
+		)
+		(pin "25"
+		)
+		(pin "10"
+		)
+		(pin "20"
+		)
+		(pin "22"
+		)
+		(pin "2"
+		)
+		(pin "19"
+		)
+		(pin "11"
+		)
+		(pin "9"
+		)
+		(pin "3"
 		)
 		(pin "5"
 		)
-		(pin "3"
-		)
-		(pin "19"
-		)
-		(pin "4"
-		)
-		(pin "16"
-		)
-		(pin "9"
-		)
-		(pin "12"
-		)
-		(pin "13"
-		)
-		(pin "10"
-		)
-		(pin "11"
-		)
-		(pin "17"
-		)
-		(pin "15"
-		)
-		(pin "14"
-		)
-		(pin "20"
-		)
-		(pin "8"
-		)
-		(pin "1"
+		(pin "26"
 		)
 		(instances
