File: CoolPackReceiver/HW/KiCAD/CoolPack/CoolPack.kicad_sch (KiCad schematic)
At the start: 2 parts, among them U1 nRF24L01P, U2 STM32U595RJTxQ

Commit message: Clean start
Other:
- note added: "AUDIO CoDec TLV320DAC3203IYZKR"
Changed lines of the file:
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@@
 	(generator_version "9.0")
 	(paper "A4")
+	(text "AUDIO CoDec TLV320DAC3203IYZKR"
+		(exclude_from_sim no)
+		(at 242.316 34.29 0)
+		(effects
+			(font
+				(size 1.27 1.27)
+			)
+		)
+	)
 	(symbol
 		(lib_id "MCU_ST_STM32U5:STM32U595RJTxQ")
