File: CoolPackReceiver/HW/KiCAD/CoolPack.kicad_pcb (KiCad board)
At the start: 2 copper layers, 0 parts

Commit message: CoolPack : rooting wip
Parts:
- added AE401: Antenna, Custom:Antenna, F.Cu at (92.3, 102.6)
- added BT101: Battery_Cell, Connector_JST:JST_PH_S2B-PH-K_1x02_P2.00mm_Horizontal, B.Cu at (93.9, 120.2)
- added C101: 4u7, Capacitor_SMD:C_0603_1608Metric, F.Cu at (75.1, 121.2)
- added C102: 4u7, Capacitor_SMD:C_0603_1608Metric, F.Cu at (133.7, 135.3)
- added C103: 1u, Capacitor_SMD:C_0603_1608Metric, F.Cu at (75.1, 126.2)
- added C104: 1u, Capacitor_SMD:C_0603_1608Metric, F.Cu at (75.1, 128.8)
- added C105: 1u, Capacitor_SMD:C_0402_1005Metric, F.Cu at (78.5, 128.0)
- added C106: 1u, Capacitor_SMD:C_0402_1005Metric, F.Cu at (78.5, 130.0)
- added C201: 1u, Capacitor_SMD:C_0402_1005Metric, F.Cu at (59.4, 103.8)
- added C202: 100n, Capacitor_SMD:C_0402_1005Metric, F.Cu at (59.4, 105.8)
- added C203: 4.7p, Capacitor_SMD:C_0402_1005Metric, F.Cu at (59.4, 107.7)
- added C204: 4.7p, Capacitor_SMD:C_0402_1005Metric, F.Cu at (59.4, 109.7)
- added C205: 10u, Capacitor_SMD:C_0805_2012Metric, F.Cu at (66.3, 99.9)
- added C206: 100n, Capacitor_SMD:C_0402_1005Metric, F.Cu at (59.4, 111.7)
- added C207: 100n, Capacitor_SMD:C_0402_1005Metric, F.Cu at (59.4, 113.6)
- added C208: 100n, Capacitor_SMD:C_0402_1005Metric, F.Cu at (62.3, 103.8)
- added C209: 100n, Capacitor_SMD:C_0402_1005Metric, F.Cu at (62.3, 105.8)
- added C210: 4u7, Capacitor_SMD:C_0402_1005Metric, F.Cu at (62.3, 107.7)
- added C211: 4u7, Capacitor_SMD:C_0402_1005Metric, F.Cu at (62.3, 109.7)
- added C212: 100n, Capacitor_SMD:C_0402_1005Metric, F.Cu at (62.3, 111.7)
- added C301: 10u, Capacitor_SMD:C_0805_2012Metric, F.Cu at (60.9, 118.9)
- added C302: 100n, Capacitor_SMD:C_0402_1005Metric, F.Cu at (57.2, 118.4)
- added C303: 1u, Capacitor_SMD:C_0402_1005Metric, F.Cu at (57.2, 120.3)
- added C304: 1u, Capacitor_SMD:C_0402_1005Metric, F.Cu at (57.2, 122.3)
- added C305: 100n, Capacitor_SMD:C_0402_1005Metric, F.Cu at (57.2, 124.3)
- added C306: 1u, Capacitor_SMD:C_0402_1005Metric, F.Cu at (57.2, 126.2)
- added C307: 47u, Capacitor_SMD:C_0805_2012Metric, F.Cu at (80.3, 137.0)
- added C308: 47u, Capacitor_SMD:C_0805_2012Metric, F.Cu at (60.9, 124.9)
- added C401: 47u, Capacitor_SMD:C_0805_2012Metric, F.Cu at (82.8, 106.0)
- added C402: 100n, Capacitor_SMD:C_0402_1005Metric, F.Cu at (75.3, 91.6)
- added C403: 100n, Capacitor_SMD:C_0402_1005Metric, F.Cu at (75.3, 93.5)
- added C404: 100n, Capacitor_SMD:C_0402_1005Metric, F.Cu at (75.3, 95.5)
- added C405: 33n, Capacitor_SMD:C_0402_1005Metric, F.Cu at (75.3, 97.5)
- added C406: 4.7p, Capacitor_SMD:C_0402_1005Metric, F.Cu at (75.3, 99.5)
- added C407: 2.2n, Capacitor_SMD:C_0402_1005Metric, F.Cu at (78.2, 91.6)
- added C408: 4.7p, Capacitor_SMD:C_0402_1005Metric, F.Cu at (78.2, 93.5)
- added C409: 4.7p, Capacitor_SMD:C_0402_1005Metric, F.Cu at (78.2, 95.5)
- added C410: 1.5p, Capacitor_SMD:C_0402_1005Metric, F.Cu at (118.3, 94.0)
- added C411: 1.5p, Capacitor_SMD:C_0402_1005Metric, F.Cu at (90.6, 106.3)
- added D101: LED, LED_SMD:LED_0603_1608Metric, F.Cu at (133.7, 130.2)
- added IC101: MCP73831-2ACI_MC, Custom:SON50P300X200X100-9N-D, F.Cu at (138.0, 127.4)
- added IC102: AP7345D-1833RH4-7, Custom:AP7345D1833RH47, F.Cu at (82.5, 124.8)
- added IC301: TLV320DAC3203IRGET, Custom:QFN50P400X400X100-25N-D, F.Cu at (96.2, 129.8)
- added J1: AudioJack4_SwitchTR1, Connector_Audio:Jack_3.5mm_PJ31060-I_Horizontal, B.Cu at (95.4, 141.2)
- added L201: 39nH, Inductor_SMD:L_0402_1005Metric, F.Cu at (65.2, 103.8)
- added L202: 2u2, Inductor_SMD:L_1008_2520Metric, F.Cu at (66.5, 96.5)
- added L401: 2.7nH, Inductor_SMD:L_0402_1005Metric, F.Cu at (112.5, 88.1)
- added L402: 8.2nH, Inductor_SMD:L_0402_1005Metric, F.Cu at (112.5, 90.1)
- added L403: 3.9nH, Inductor_SMD:L_0402_1005Metric, F.Cu at (112.5, 92.1)
- added R101: 470k, Resistor_SMD:R_0402_1005Metric, F.Cu at (137.1, 132.5)
- added R102: 1k8, Resistor_SMD:R_0402_1005Metric, F.Cu at (137.1, 139.1)
- added R201: 5k1, Resistor_SMD:R_0402_1005Metric, F.Cu at (116.1, 109.9)
- added R202: 5k1, Resistor_SMD:R_0402_1005Metric, F.Cu at (116.1, 104.0)
- added R203: 100k, Resistor_SMD:R_0402_1005Metric, F.Cu at (65.2, 109.8)
- added R401: 22k, Resistor_SMD:R_0402_1005Metric, F.Cu at (72.5, 97.6)
- added R402: 1M, Resistor_SMD:R_0402_1005Metric, F.Cu at (72.5, 99.5)
- added TP201: TestPoint_Small, TestPoint:TestPoint_Pad_D1.0mm, F.Cu at (59.5, 92.1)
- added TP202: TestPoint_Small, TestPoint:TestPoint_Pad_D1.0mm, F.Cu at (59.5, 95.2)
- added TP203: TestPoint_Small, TestPoint:TestPoint_Pad_D1.0mm, F.Cu at (59.5, 98.2)
- added TP204: TestPoint_Small, TestPoint:TestPoint_Pad_D1.0mm, F.Cu at (102.0, 95.8)
- added TP205: TestPoint_Small, TestPoint:TestPoint_Pad_D1.0mm, F.Cu at (62.5, 92.1)
- added TP206: TestPoint_Small, TestPoint:TestPoint_Pad_D1.0mm, F.Cu at (62.5, 95.2)
- added TP207: TestPoint_Small, TestPoint:TestPoint_Pad_D1.0mm, F.Cu at (61.9, 97.4)
- added U201: STM32U595RJTxQ, Package_QFP:LQFP-64_10x10mm_P0.5mm, F.Cu at (110.0, 124.1)
- added U202: USBLC6-2SC6, Package_TO_SOT_SMD:SOT-23-6, F.Cu at (114.4, 107.0)
- added U401: nRF24L01P, Package_DFN_QFN:QFN-20-1EP_4x4mm_P0.5mm_EP2.5x2.5mm, F.Cu at (104.6, 105.2)
- added USB/Charge: USB_C_Receptacle_USB2.0_16P, Connector_USB:USB_C_Receptacle_XKB_U262-16XN-4BVC11, F.Cu at (122.8, 107.0)
- added Y201: 16 MHz, Custom:CX3225FB16000B0FZZH1, F.Cu at (52.5, 125.5)
- added Y401: 16 MHz, Custom:CX3225FB16000B0FZZH1, F.Cu at (78.7, 111.4)
Routing:
- net /MCU/USBC_D-: track 0.00 -> 6.11 mm
- net /MCU/USBC_D+: track 0.00 -> 5.63 mm
- net /MCU/USB_CC1: track 0.00 -> 3.42 mm
- net /MCU/USB_CC2: track 0.00 -> 3.34 mm
- net GND: track 0.00 -> 2.41 mm, vias 0 -> 21
- net /RF/Antenna_Feed: track 0.00 -> 1.36 mm
- net VBUS: track 0.00 -> 1.18 mm, vias 0 -> 7
- added copper zone on F.Cu, net /RF/Antenna_Feed
- added copper zone on B.Cu, net GND
- added copper zone on F.Cu, net GND
- added copper zone on In1.Cu, net GND
- added copper zone on F.Cu, net VBUS
- added copper zone on In2.Cu, net VBUS
Other:
- board outline added: 38 x 49 mm
- copper layers 2 -> 4
