File: CoolPackReceiver/HW/KiCAD/CoolPack.kicad_sch (KiCad schematic)
At the start: 12 parts, among them IC101 MCP73831-2ACI_MC, IC102 AP7345D-1833RH4-7

Commit message: CoolPack : rooting wip
Other:
- note added: "check if shottky or is possible between the batt+ and VBUS for LDO supply"
- note removed: "check if shotky or is possible between the batt+ and VBUS for LDO supply"
Changed lines of the file:
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@@
 		(rev "V0.1")
 	)
-	(text "check if shotky or is possible between the batt+ and VBUS for LDO supply"
+	(text "check if shottky or is possible between the batt+ and VBUS for LDO supply"
 		(exclude_from_sim no)
 		(at 153.162 50.546 0)
